File: hardware/kicad/synthy/synthy.kicad_sch (KiCad schematic)
At the start: 0 parts

Commit message: finished schematic+ routing
Parts:
- added C1, C10: 10nF, Capacitor_THT:C_Disc_D5.0mm_W2.5mm_P5.00mm, symbol Device:C
- added C11: 4.7nF, Capacitor_THT:C_Disc_D5.0mm_W2.5mm_P5.00mm, symbol Device:C
- added C12: 1µF, Capacitor_THT:C_Disc_D5.0mm_W2.5mm_P5.00mm, symbol Device:C
- added C13, C3: 100µF, Capacitor_THT:CP_Radial_D6.3mm_P2.50mm, symbol Device:C_Polarized
- added C14, C4, C5, C7, C8: 100nF, Capacitor_THT:C_Disc_D5.0mm_W2.5mm_P5.00mm, symbol Device:C
- added C15, C6: 10µF, Capacitor_THT:CP_Radial_D5.0mm_P2.00mm, symbol Device:C_Polarized
- added C16: 47nF, Capacitor_THT:C_Disc_D5.0mm_W2.5mm_P5.00mm, symbol Device:C
- added C17: 220µF, Capacitor_THT:CP_Radial_D8.0mm_P3.50mm, symbol Device:C_Polarized
- added C9: 47nF, Capacitor_THT:C_Rect_L7.2mm_W2.5mm_P5.00mm_FKS2_FKP2_MKS2_MKP2, symbol Device:C
- added D10, D12, D14, D16, D18, D2, D4, D6, D8: LED, LED_THT:LED_D3.0mm, symbol Device:LED
- added D11, D13, D15, D17, D19, D5, D7, D9: 1N4148, Diode_THT:D_DO-35_SOD27_P2.54mm_Vertical_AnodeUp, symbol Diode:1N4148
- added J1: USB_C_Receptacle_PowerOnly_6P, Connector_USB:USB_C_Receptacle_GCT_USB4125-xx-x-0190_6P_TopMnt_Horizontal, symbol Connector:USB_C_Receptacle_PowerOnly_6P
- added J2: Conn_01x02, Connector_JST:JST_PH_B2B-PH-K_1x02_P2.00mm_Vertical, symbol Connector_Generic:Conn_01x02
- added R10: 47k, Resistor_THT:R_Axial_DIN0207_L6.3mm_D2.5mm_P10.16mm_Horizontal, symbol Device:R
- added R11, R13, R15, R17, R19, R21, R23, R25: 2.2k, Resistor_THT:R_Axial_DIN0207_L6.3mm_D2.5mm_P2.54mm_Vertical, symbol Device:R
- added R12, R14, R16, R18, R20, R22, R24, R26: 10k, Resistor_THT:R_Axial_DIN0207_L6.3mm_D2.5mm_P2.54mm_Vertical, symbol Device:R
- added R2, R3: 5.1k, Resistor_THT:R_Axial_DIN0207_L6.3mm_D2.5mm_P10.16mm_Horizontal, symbol Device:R
- added R27, R7: 4.7k, Resistor_THT:R_Axial_DIN0207_L6.3mm_D2.5mm_P10.16mm_Horizontal, symbol Device:R
- added R28: 10, Resistor_THT:R_Axial_DIN0207_L6.3mm_D2.5mm_P10.16mm_Horizontal, symbol Device:R
- added R4, R6: 1k, Resistor_THT:R_Axial_DIN0207_L6.3mm_D2.5mm_P10.16mm_Horizontal, symbol Device:R
- added R5: 10k, Resistor_THT:R_Axial_DIN0207_L6.3mm_D2.5mm_P10.16mm_Horizontal, symbol Device:R
- added R8: 100k, Resistor_THT:R_Axial_DIN0207_L6.3mm_D2.5mm_P10.16mm_Horizontal, symbol Device:R
- added R9: 2.2k, Resistor_THT:R_Axial_DIN0207_L6.3mm_D2.5mm_P10.16mm_Horizontal, symbol Device:R
- added RV1: A100k, Potentiometer_THT:Potentiometer_Alps_RK09K_Single_Vertical, symbol Device:R_Potentiometer
- added RV10, RV2, RV3, RV4, RV5, RV6, RV7, RV8, RV9: B100k, Potentiometer_THT:Potentiometer_Alps_RK09K_Single_Vertical, symbol Device:R_Potentiometer
- added RV11: B50k, Potentiometer_THT:Potentiometer_Alps_RK09K_Single_Vertical, symbol Device:R_Potentiometer
- added SW1: SW_DIP_x08, Button_Switch_THT:SW_DIP_SPSTx08_Slide_9.78x22.5mm_W7.62mm_P2.54mm, symbol Switch:SW_DIP_x08
- added SW2, SW3: SW_SPDT, Button_Switch_THT:SW_Slide_SPDT_Straight_CK_OS102011MS2Q, symbol Switch:SW_SPDT
- added U1, U4: LMC555CN, Package_DIP:DIP-8_W7.62mm_Socket, symbol Timer:TLC555xP
- added U2: 74HC4017, Package_DIP:DIP-16_W7.62mm_Socket, symbol 4xxx:4017
- added U3: LM386, Package_DIP:DIP-8_W7.62mm_Socket, symbol Amplifier_Audio:LM386
Connections:
- new net: D2.2 (A), R4.2
- new net: RV1.2, U3.3 (+)
- new net: C12.2, RV1.3
- new net: R16.1, RV5.1, RV5.2
- new net: C9.1, R9.2, U4.2 (TRIG), U4.6 (THRES)
- new net: R14.1, RV4.1, RV4.2
- new net: D7.2 (A), R14.2
- new net: C10.1, U4.5 (CONT)
- new net: R22.1, RV8.1, RV8.2
- new net: D15.2 (A), R22.2
- new net: C6.1, R7.2, U1.2 (TRIG), U1.6 (THRES)
- new net: R5.2, SW2.2 (B), U1.4 (~{RST})
- new net: C1.1, U1.5 (CONT)
- new net: R7.1, RV2.1, RV2.2, U1.7 (DISCH)
- new net: D14.2 (A), R21.2
- new net: D17.2 (A), R24.2
- new net: D10.2 (A), R17.2
- new net: D4.2 (A), R11.2
- new net: C15.1, U3.7 (BYPASS)
- new net: R12.1, RV3.1, RV3.2
- new net: R18.1, RV6.1, RV6.2
- new net: R26.1, RV10.1, RV10.2
- new net: D19.2 (A), R26.2
- new net: R10.1, U4.3 (OUT)
- new net: C17.1, R28.1, U3.5
- new net: C17.2, J2.1 (Pin_1)
- new net: D6.2 (A), R13.2
- new net: R24.1, RV9.1, RV9.2
- new net: D18.2 (A), R25.2
- new net: D16.2 (A), R23.2
- new net: J1.A5 (CC1), R2.1
- new net: D11.2 (A), R18.2
- new net: R6.1, RV2.3
- new net: D5.2 (A), R12.2
- new net: D13.2 (A), R20.2
- new net: C16.1, R28.2
- new net: R8.1, SW3.2 (B), U2.15 (Reset)
- new net: D12.2 (A), R19.2
- new net: J1.B5 (CC2), R3.1
- new net: D8.2 (A), R15.2
- new net: SW3.1 (A), U2.9 (Q8)
- new net: D9.2 (A), R16.2
- new net: R20.1, RV7.1, RV7.2
- new net +5V: C13.1, C14.1, C3.1, C4.1, C5.1, C7.2, C8.2, J1.A9 (VBUS), J1.B9 (VBUS), R4.1, R5.1, R6.2, U1.8 (VCC), U2.16 (VDD), U3.6 (V+), U4.4 (~{RST}), U4.8 (VCC)
- new net A: R10.2, R27.1, RV11.3
- new net B: C11.2, C12.1, RV11.1, RV11.2
- new net CLK: U1.3 (OUT), U2.14 (CLK)
- new net GND: C1.2, C10.2, C11.1, C13.2, C14.2, C15.2, C16.2, C3.2, C4.2, C5.2, C6.2, C7.1, C8.1, C9.2, D10.1 (K), D12.1 (K), D14.1 (K), D16.1 (K), D18.1 (K), D2.1 (K), D4.1 (K), D6.1 (K), D8.1 (K), J1.A12 (GND), J1.B12 (GND), J1.SH (SHIELD), J2.2 (Pin_2), R2.2, R27.2, R3.2, R8.2, RV1.1, SW2.1 (A), U1.1 (GND), U2.13 (CKEN), U2.8 (VSS), U3.2 (-), U3.4 (GND), U4.1 (GND)
- new net Q0: R11.1, SW1.1, U2.3 (Q0)
- new net Q1: R15.1, SW1.2, U2.2 (Q1)
- new net Q2: R19.1, SW1.3, U2.4 (Q2)
- new net Q3: R23.1, SW1.4, U2.7 (Q3)
- new net Q4: R13.1, SW1.5, SW3.3 (C), U2.10 (Q4)
- new net Q5: R17.1, SW1.6, U2.1 (Q5)
- new net Q6: R21.1, SW1.7, U2.5 (Q6)
- new net Q7: R25.1, SW1.8, U2.6 (Q7)
- new net S0: RV3.3, SW1.16
- new net S1: RV5.3, SW1.15
- new net S2: RV7.3, SW1.14
- new net S3: RV9.3, SW1.13
- new net S4: RV4.3, SW1.12
- new net S5: RV6.3, SW1.11
- new net S6: RV8.3, SW1.10
- new net S7: RV10.3, SW1.9
- new net TONE_RC: D11.1 (K), D13.1 (K), D15.1 (K), D17.1 (K), D19.1 (K), D5.1 (K), D7.1 (K), D9.1 (K), R9.1, U4.7 (DISCH)
- no-connect marks 0 -> 5
Other:
- title: (none) -> Synthy
